File: pcb-using-pico/psion-org2-main/file612F7BBD.sch (KiCad schematic (older format))
At the start: 36 parts

Commit message: Schematic updates
Parts:
- gave numbers to parts that had none: 36

Commit message: PCB updates
Parts:
- SW1: value sw -> AC_ON
- SW10: value sw -> n
- SW11: value sw -> t
- SW12: value sw -> del
- SW13: value sw -> up
- SW14: value sw -> c
- SW15: value sw -> i
- SW16: value sw -> o
- SW17: value sw -> u
- SW18: value sw -> y
- SW19: value sw -> down
- SW2: value sw -> A
- SW20: value sw -> d
- SW21: value sw -> j
- SW22: value sw -> p
- SW23: value sw -> v
- SW24: value sw -> z
- SW25: value sw -> left
- SW26: value sw -> e
- SW27: value sw -> k
- SW28: value sw -> q
- SW29: value sw -> w
- SW3: value sw -> g
- SW30: value sw -> spc
- SW31: value sw -> right
- SW32: value sw -> f
- SW33: value sw -> L
- SW34: value sw -> r
- SW35: value sw -> x
- SW36: value sw -> exe
- SW4: value sw -> m
- SW5: value sw -> s
- SW6: value sw -> shft
- SW7: value sw -> mode
- SW8: value sw -> b
- SW9: value sw -> h
Connections:
- net KC0 renamed K2
- net K2: no longer SW1.2 (B)
- net KC1 renamed K3
- net KC2 renamed K4
- net KC3 renamed K7
- net KC4 renamed K5
- net KC5 renamed K6
- net KR0 renamed K1
- net K1: no longer SW1.1 (A)
- net KR1 renamed P56
- net KR2 renamed P55
- net KR3 renamed P54
- net KR4 renamed p53
- net KR5 renamed P52
- new net +3V3: SW1.1 (A)
- new net P57: SW1.2 (B)
