File: pcb-using-pico/psion-org2-main/psion-org2-main.sch (KiCad schematic (older format))
At the start: 32 parts, among them J2 Conn_02x08_Odd_Even, J3 Conn_01x03_Female, U10 74LS245, U9 74LS245

Commit message: Updates to control PCB schematic
Parts:
- added C?: 4u7 25V, symbol Device:C_Small
- added C?: 4u7, symbol Device:C_Small
- added C?: 100nF, symbol Device:C_Small
- added J?: Conn_01x24_Female, symbol Connector:Conn_01x24_Female
- added R?: 910k, symbol Device:R_Small
- added R? (x2): 10k, symbol Device:R_Small
Connections:
- net labels added: KR0, KR1, KR2, KR3, KR4, KR5, LATCHIN, OLED_RES, OLED_SCL, OLED_SDA, SCLKIN, SDAIN
- wire segments 113 -> 202
Other:
- moved on the sheet: J2, R?

Commit message: More updates
Parts:
- removed D?: SS36, Diode_SMD:D_SOD-123, symbol fx502-recreate-rescue:DIODE-Microtan_65_CPU-cache
- added C? (x2): C, Capacitor_SMD:C_0805_2012Metric_Pad1.15x1.40mm_HandSolder, symbol Device:C
- added R? (x2): 4k7, Resistor_SMD:R_0805_2012Metric, symbol Device:R_Small
- added U?: MCP7940N-xSN, Package_SO:SO-8_3.9x4.9mm_P1.27mm, symbol Timer:MCP7940N-xSN
- added Y?: 32k768Hz, Crystal:Crystal_SMD_3215-2Pin_3.2x1.5mm, symbol Device:Crystal
- D?: value D -> SS36
Connections:
- net labels added: MISO, MOSI, RTC_MFP, RTC_SCL, RTC_SDA, VBAT
- wire segments 202 -> 230
Other:
- note removed: "Check transistor pinout footprint"
- moved on the sheet: J2

Commit message: Schematic updates
Parts:
- removed C6, C7: 100n, Capacitor_SMD:C_0402_1005Metric, symbol Device:C
- removed C8: 1u, Capacitor_SMD:C_0402_1005Metric, symbol Device:C
- removed R? (x4): R_Small, symbol Device:R_Small
- added C11, C12, C9: 100n, Capacitor_SMD:C_0402_1005Metric, symbol Device:C
- added J3: Conn_01x27_Female, symbol Connector:Conn_01x27_Female
- added R6, R7, R8, R9: 100k, symbol Device:R_Small
- R1: renamed from R?; value R_Small -> 10k
- R5: renamed from R?; value R_Small -> 100k
- gave numbers to parts that had none: 26
- renumbered C10 to C5, C14 to C6, C15 to C7, C16 to C8, J3 to J2, J2 to J4, U9 to U6, U10 to U7
Connections:
- net labels added: KC0, KC1, KC2, KC3, KC4, KC5, VOLED
- net labels removed: +1V1, VPP
- wire segments 230 -> 238
Other:
- note added: "KR0 used for power on"
- note removed: "Make sure C10 is close to pin 44 of RP2040"
- note removed: "Make sure C8 is close to pin 45 of RP2040"
- moved on the sheet: C1, C2, C3, C5, C6, C7, C8, J1, J2, J4, R1, R2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

Commit message: Added start of code for main board replacement. Wifi server
Parts:
- removed J4: Conn_02x08_Odd_Even, psion_org_2:Psion_datapak_2x08_P2.54mm_Horizontal, symbol Connector_Generic:Conn_02x08_Odd_Even
Connections:
- wire segments 238 -> 239
Changed lines of the file:
@@
 Wire Wire Line
 	9300 1800 9300 1850
-Text GLabel 15575 -1875 0    50   Input ~ 0
+Text GLabel 4200 8150 2    50   Input ~ 0
 SD1
-Text GLabel 15575 -1975 0    50   Input ~ 0
+Text GLabel 4200 8350 2    50   Input ~ 0
 SD3
-Text GLabel 15575 -2075 0    50   Input ~ 0
+Text GLabel 4200 8550 2    50   Input ~ 0
 SD5
-Text GLabel 15575 -2175 0    50   Input ~ 0
+Text GLabel 4200 8750 2    50   Input ~ 0
 SD7
-Text GLabel 15575 -2275 0    50   Input ~ 0
+Text GLabel 4200 9250 2    50   Input ~ 0
 SMR
-Text GLabel 15575 -2375 0    50   Input ~ 0
+Text GLabel 4200 9150 2    50   Input ~ 0
 SOE
-Wire Wire Line
-	15075 -2475 15575 -2475
-Text GLabel 16075 -2475 2    50   Input ~ 0
+Text GLabel 4200 8850 2    50   Input ~ 0
 SPGM
-Text GLabel 16075 -2375 2    50   Input ~ 0
+Text GLabel 4200 8950 2    50   Input ~ 0
 SS
-Text GLabel 16075 -2275 2    50   Input ~ 0
+Text GLabel 4200 9050 2    50   Input ~ 0
 SCLK
-Text GLabel 16075 -1875 2    50   Input ~ 0
+Text GLabel 4200 8050 2    50   Input ~ 0
 SD0
-Text GLabel 16075 -2175 2    50   Input ~ 0
+Text GLabel 4200 8650 2    50   Input ~ 0
 SD6
-Text GLabel 16075 -2075 2    50   Input ~ 0
+Text GLabel 4200 8450 2    50   Input ~ 0
 SD4
-Text GLabel 16075 -1975 2    50   Input ~ 0
+Text GLabel 4200 8250 2    50   Input ~ 0
 SD2
 $Comp
 L power:GND #PWR?
 U 1 1 61058D25
-P 15075 -1825
+P 4925 7950
 AR Path="/6104FF77/61058D25" Ref="#PWR?"  Part="1"
 AR Path="/61058D25" Ref="#PWR025"  Part="1"
-F 0 "#PWR025" H 15075 -2075 50  0001 C CNN
-F 1 "GND" H 15075 -2000 50  0000 C CNN
-F 2 "" H 15075 -1825 50  0001 C CNN
-F 3 "" H 15075 -1825 50  0001 C CNN
-	1    15075 -1825
-	1    0    0    -1
-$EndComp
-$Comp
-L Connector_Generic:Conn_02x08_Odd_Even J?
-U 1 1 6133A2AE
-P 15775 -2275
-AR Path="/6104FF77/6133A2AE" Ref="J?"  Part="1"
-AR Path="/6133A2AE" Ref="J4"  Part="1"
-F 0 "J4" H 15825 -1758 50  0000 C CNN
-F 1 "Conn_02x08_Odd_Even" H 15825 -1849 50  0000 C CNN
-F 2 "psion_org_2:Psion_datapak_2x08_P2.54mm_Horizontal" H 15775 -2275 50  0001 C CNN
-F 3 "~" H 15775 -2275 50  0001 C CNN
-	1    15775 -2275
-	1    0    0    -1
-$EndComp
-Wire Wire Line
-	15075 -2475 15075 -1825
+F 0 "#PWR025" H 4925 7700 50  0001 C CNN
+F 1 "GND" H 4925 7775 50  0000 C CNN
+F 2 "" H 4925 7950 50  0001 C CNN
+F 3 "" H 4925 7950 50  0001 C CNN
+	1    4925 7950
+	1    0    0    -1
+$EndComp
 $Comp
 L Connector:Conn_01x03_Female J2
@@
 L power:+3V3 #PWR05
 U 1 1 61672821
-P 2125 7950
-F 0 "#PWR05" H 2125 7800 50  0001 C CNN
-F 1 "+3V3" H 2140 8123 50  0000 C CNN
-F 2 "" H 2125 7950 50  0001 C CNN
-F 3 "" H 2125 7950 50  0001 C CNN
-	1    2125 7950
+P 5000 10475
+F 0 "#PWR05" H 5000 10325 50  0001 C CNN
+F 1 "+3V3" H 5015 10648 50  0000 C CNN
+F 2 "" H 5000 10475 50  0001 C CNN
+F 3 "" H 5000 10475 50  0001 C CNN
+	1    5000 10475
 	1    0    0    -1
 $EndComp
@@
 	1    0    0    -1
 $EndComp
+Wire Wire Line
+	4200 7950 4925 7950
+Wire Wire Line
+	5000 10550 5000 10475
+Wire Wire Line
+	4200 10550 5000 10550
 $EndSCHEMATC

Commit message: PCB updates
Parts:
- added R? (x3): 100k, symbol Device:R_Small
Connections:
- net labels added: K1, K2, K3, K4, K5, K6, K7, P50, P51, P52, P53, P54, P55, P56, P57
- net labels removed: KC0, KC1, KC2, KC3, KC4, KC5, KR0, KR1, KR2, KR3, KR4, KR5
- wire segments 239 -> 254
Other:
- moved on the sheet: C10, C13, C14, C4, D1, JP1, L1, R10, R11, R12, R13, R14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

Commit message: Last commit before splitting to two PCBs
Parts:
- added C17, C18, C19, C20: C_Small, Capacitor_SMD:C_0805_2012Metric, symbol Device:C_Small
- added C21: 10uF, Capacitor_SMD:C_1210_3225Metric_Pad1.42x2.65mm_HandSolder, symbol Device:C_Small
- added C22: 100nF, Capacitor_SMD:C_0805_2012Metric, symbol Device:C_Small
- added R22, R23: R_Small, Resistor_SMD:R_0805_2012Metric, symbol Device:R_Small
- added U10, U11: AMS1117-3.3, Package_TO_SOT_SMD:SOT-223-3_TabPin2, symbol pak_breakout:AMS1117-3.3
- C1, C2, C3: footprint (none) -> Capacitor_SMD:C_0805_2012Metric
- C11, C12, C5, C6, C7, C8, C9: footprint Capacitor_SMD:C_0402_1005Metric -> Capacitor_SMD:C_0805_2012Metric
- C13, C14: footprint Capacitor_SMD:C_0805_2012Metric_Pad1.15x1.40mm_HandSolder -> Capacitor_SMD:C_0805_2012Metric
- R1, R2, R3, R4, R5, R6, R7, R8, R9: footprint (none) -> Resistor_SMD:R_0805_2012Metric
- R10, R11, R12: footprint Resistor_SMD:R_0805_2012Metric_Pad1.15x1.40mm_HandSolder -> Resistor_SMD:R_0805_2012Metric
- R15: footprint Capacitor_SMD:C_0402_1005Metric -> Resistor_SMD:R_0805_2012Metric
- R19, R20, R21: renamed from R?; footprint (none) -> Resistor_SMD:R_0805_2012Metric
Connections:
- net +3V3: now also C1.1, C3.1, J1.5 (Pin_5), J1.6 (Pin_6), R3.1, R4.1
- net GND: now also U1.28 (GND), C17.2, C18.2, C19.2, C20.2, R23.2, U10.1 (GND), U11.1 (GND); no longer R3.2, R4.2
- net OLED_SCL: now also R3.2; no longer R3.1
- net OLED_SDA: now also R4.2; no longer R4.1
- net VBAT: now also J3.26 (Pin_26), C17.1, C18.1, R22.1, U10.3 (VI), U11.3 (VI); no longer U5.3 (VBAT)
- net VOLED: now also C21.1, C22.1
- net at C10.2, C4.2, R10.2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: now also C21.2, C22.2
- new net: R22.2, R23.1, U5.3 (VBAT)
- new net VccESP: C20.1, U11.2 (VO)
- new net VccPico: C19.1, U10.2 (VO)
Other:
- note added: "850nA 1300mV\n1200nA 3000mV\n9000nA 5500mV\n"
- note added: "ER-OLED022-1"
- note added: "Supply Current:\nESP-WROOM: 500mA\nPico: 150mA\nOLED display: \n"
- moved on the sheet: C1, C13, C14, C3, R13, R14, R3, R4, U5, Y1
