File: pcb-using-pico/psion-org2-main/psion-org2-main.sch (KiCad schematic (older format))
At the start: 83 parts, among them J1 Conn_01x24_Female, J2 Conn_01x03_Female, J3 Conn_01x27_Female, J4 Conn_01x02_Female, J5 Conn_01x02_Female, J6 Conn_01x11_Female, M1 P-CH-MOSFET, M2 P-CHANNEL-MOSFET, M3 P-CHANNEL-MOSFET, U1 Pico, U10 AMS1117-3.3, U2 74HC595, U3 Regulator_Switching_MT3608, U4 74LS165, U5 74HC595, U7 MCP7940N-xSN, Y1 32k768Hz

Commit message: V1.1 PCBs
Parts:
- removed JP3, JP5, JP7: Jumper_NO_Small, Jumper:SolderJumper-2_P1.3mm_Open_RoundedPad1.0x1.5mm, symbol Device:Jumper_NO_Small
- C5: value C_Small -> 100nF
Connections:
- net DRV_HV: no longer names the net of U5.15 (QA)
Changed lines of the file:
@@
 Wire Wire Line
 	10100 8925 10700 8925
-Text GLabel 6325 1150 2    50   Input ~ 0
-DRV_HV
 $Comp
 L Device:R_Small R1
@@
 Wire Wire Line
 	1625 1250 1625 1425
-Text GLabel 11075 7525 0    50   Input ~ 0
-VBAT
 Text GLabel 6325 1450 2    50   Input ~ 0
 5V_ON
@@
 	1    0    0    -1
 $EndComp
-$Comp
-L Device:Jumper_NO_Small JP3
-U 1 1 6194B084
-P 8275 8625
-F 0 "JP3" H 8275 8810 50  0000 C CNN
-F 1 "Jumper_NO_Small" H 8275 8719 50  0000 C CNN
-F 2 "Jumper:SolderJumper-2_P1.3mm_Open_RoundedPad1.0x1.5mm" H 8275 8625 50  0001 C CNN
-F 3 "~" H 8275 8625 50  0001 C CNN
-	1    8275 8625
-	1    0    0    -1
-$EndComp
 Wire Wire Line
 	7775 8300 7775 8350
@@
 Wire Wire Line
 	8375 8350 8700 8350
-Wire Wire Line
-	8700 8350 8700 8625
-Wire Wire Line
-	8375 8625 8700 8625
-Connection ~ 8700 8625
-Wire Wire Line
-	8700 8625 8700 8925
-Text GLabel 7775 8625 0    50   Input ~ 0
-VBAT
-Wire Wire Line
-	7775 8625 8175 8625
 $Comp
 L GeekAmmo:P-CHANNEL-MOSFET M1
@@
 	1    0    0    -1
 $EndComp
-$Comp
-L Device:Jumper_NO_Small JP5
-U 1 1 61A42C08
-P 11425 7525
-F 0 "JP5" H 11425 7710 50  0000 C CNN
-F 1 "Jumper_NO_Small" H 11425 7619 50  0000 C CNN
-F 2 "Jumper:SolderJumper-2_P1.3mm_Open_RoundedPad1.0x1.5mm" H 11425 7525 50  0001 C CNN
-F 3 "~" H 11425 7525 50  0001 C CNN
-	1    11425 7525
-	1    0    0    -1
-$EndComp
-Wire Wire Line
-	11075 7525 11325 7525
 Text GLabel 12125 7525 2    50   Input ~ 0
 VBAT_SWITCHED1
 Wire Wire Line
-	11525 7525 11950 7525
-Wire Wire Line
 	11525 7225 11950 7225
 Wire Wire Line
 	11950 7225 11950 7525
-Connection ~ 11950 7525
 Wire Wire Line
 	11950 7525 12125 7525
@@
 Wire Wire Line
 	9000 6575 9000 7075
-Text GLabel 11100 8175 0    50   Input ~ 0
-VBAT
 $Comp
 L Device:Jumper_NO_Small JP6
@@
 	1    0    0    -1
 $EndComp
-$Comp
-L Device:Jumper_NO_Small JP7
-U 1 1 61BE2019
-P 11450 8175
-F 0 "JP7" H 11450 8360 50  0000 C CNN
-F 1 "Jumper_NO_Small" H 11450 8269 50  0000 C CNN
-F 2 "Jumper:SolderJumper-2_P1.3mm_Open_RoundedPad1.0x1.5mm" H 11450 8175 50  0001 C CNN
-F 3 "~" H 11450 8175 50  0001 C CNN
-	1    11450 8175
-	1    0    0    -1
-$EndComp
-Wire Wire Line
-	11100 8175 11350 8175
 Text GLabel 12150 8175 2    50   Input ~ 0
 VBAT_SWITCHED2
 Wire Wire Line
-	11550 8175 11975 8175
-Wire Wire Line
 	11550 7875 11975 7875
 Wire Wire Line
 	11975 7875 11975 8175
-Connection ~ 11975 8175
 Wire Wire Line
 	11975 8175 12150 8175
@@
 P 4700 3500
 F 0 "C5" H 4792 3546 50  0000 L CNN
-F 1 "C_Small" H 4792 3455 50  0000 L CNN
+F 1 "100nF" H 4792 3455 50  0000 L CNN
 F 2 "Capacitor_SMD:C_0805_2012Metric" H 4700 3500 50  0001 C CNN
 F 3 "~" H 4700 3500 50  0001 C CNN
@@
 Text GLabel 4650 9875 2    50   Input ~ 0
 VBAT_SWITCHED1
+Wire Wire Line
+	8700 8350 8700 8925
 $EndSCHEMATC
