File: pcb-using-pico/psion-org2-main/a.sch (KiCad schematic (older format))
At the start: 59 parts

Commit message: Schematic updates
Parts:
- gave numbers to parts that had none: 58

Commit message: Last commit before splitting to two PCBs
Parts:
- C15, C16: footprint Capacitor_SMD:C_0805_2012Metric_Pad1.15x1.40mm_HandSolder -> Capacitor_SMD:C_0805_2012Metric
- R18: footprint Resistor_SMD:R_0805_2012Metric_Pad1.15x1.40mm_HandSolder -> Resistor_SMD:R_0805_2012Metric
- gave numbers to parts that had none: 1
Changed lines of the file:
@@
 F 0 "R18" V 8400 3650 50  0000 C CNN
 F 1 "390R" V 8500 3700 50  0000 C CNN
-F 2 "Resistor_SMD:R_0805_2012Metric_Pad1.15x1.40mm_HandSolder" H 8300 3700 50  0001 C CNN
+F 2 "Resistor_SMD:R_0805_2012Metric" H 8300 3700 50  0001 C CNN
 F 3 "~" H 8300 3700 50  0001 C CNN
 	1    8300 3700
@@
 DRV_HV
 $Comp
-L fx502p:SD_ebay-uSD-push_push_SMD XS?
+L fx502p:SD_ebay-uSD-push_push_SMD XS1
 U 1 1 602ED18B
 P 2275 6625
-F 0 "XS?" H 1971 6671 50  0000 R CNN
+F 0 "XS1" H 1971 6671 50  0000 R CNN
 F 1 "SD_ebay-uSD-push_push_SMD" H 1971 6580 50  0000 R CNN
 F 2 "ajm_kicad:Conn_uSDcard" H 2275 6625 10  0001 C CNN
@@
 F 0 "C15" H 5915 6246 50  0000 L CNN
 F 1 "C" H 5915 6155 50  0000 L CNN
-F 2 "Capacitor_SMD:C_0805_2012Metric_Pad1.15x1.40mm_HandSolder" H 5838 6050 50  0001 C CNN
+F 2 "Capacitor_SMD:C_0805_2012Metric" H 5838 6050 50  0001 C CNN
 F 3 "~" H 5800 6200 50  0001 C CNN
 	1    5800 6200
@@
 F 0 "C16" H 6440 6246 50  0000 L CNN
 F 1 "C" H 6440 6155 50  0000 L CNN
-F 2 "Capacitor_SMD:C_0805_2012Metric_Pad1.15x1.40mm_HandSolder" H 6363 6050 50  0001 C CNN
+F 2 "Capacitor_SMD:C_0805_2012Metric" H 6363 6050 50  0001 C CNN
 F 3 "~" H 6325 6200 50  0001 C CNN
 	1    6325 6200

Commit message: Added second connector, eeprom on power pcb
Parts:
- renumbered C15 to C18, C16 to C20, R16 to R29, R17 to R30, R18 to R31
Changed lines of the file:
@@
 Connection ~ 9350 5950
 $Comp
-L power:+3V3 #PWR028
+L power:+3V3 #PWR0118
 U 1 1 600AD885
 P 9050 1800
-F 0 "#PWR028" H 9050 1650 50  0001 C CNN
+F 0 "#PWR0118" H 9050 1650 50  0001 C CNN
 F 1 "+3V3" H 9065 1973 50  0000 C CNN
 F 2 "" H 9050 1800 50  0001 C CNN
@@
 OSCO
 $Comp
-L Device:R_Small R18
+L Device:R_Small R31
 U 1 1 6002F506
 P 8300 3700
-F 0 "R18" V 8400 3650 50  0000 C CNN
+F 0 "R31" V 8400 3650 50  0000 C CNN
 F 1 "390R" V 8500 3700 50  0000 C CNN
 F 2 "Resistor_SMD:R_0805_2012Metric" H 8300 3700 50  0001 C CNN
@@
 $EndComp
 $Comp
-L power:+3V3 #PWR026
+L power:+3V3 #PWR0119
 U 1 1 60304093
 P 2125 5875
-F 0 "#PWR026" H 2125 5725 50  0001 C CNN
+F 0 "#PWR0119" H 2125 5725 50  0001 C CNN
 F 1 "+3V3" H 2140 6048 50  0000 C CNN
 F 2 "" H 2125 5875 50  0001 C CNN
@@
 GPIO_USB_5V
 $Comp
-L power:+3V3 #PWR027
+L power:+3V3 #PWR0120
 U 1 1 605672EA
 P 4725 4775
-F 0 "#PWR027" H 4725 4625 50  0001 C CNN
+F 0 "#PWR0120" H 4725 4625 50  0001 C CNN
 F 1 "+3V3" H 4740 4948 50  0000 C CNN
 F 2 "" H 4725 4775 50  0001 C CNN
@@
 	4725 6525 4725 6175
 $Comp
-L Device:R_Small R16
+L Device:R_Small R29
 U 1 1 605ACF7F
 P 3625 5200
-F 0 "R16" H 3684 5246 50  0000 L CNN
+F 0 "R29" H 3684 5246 50  0000 L CNN
 F 1 "4k7" H 3684 5155 50  0000 L CNN
 F 2 "Resistor_SMD:R_0805_2012Metric" H 3625 5200 50  0001 C CNN
@@
 $EndComp
 $Comp
-L Device:R_Small R17
+L Device:R_Small R30
 U 1 1 605AD605
 P 3875 5200
-F 0 "R17" H 3934 5246 50  0000 L CNN
+F 0 "R30" H 3934 5246 50  0000 L CNN
 F 1 "4k7" H 3934 5155 50  0000 L CNN
 F 2 "Resistor_SMD:R_0805_2012Metric" H 3875 5200 50  0001 C CNN
@@
 	5800 6050 5800 5950
 $Comp
-L Device:C C15
+L Device:C C18
 U 1 1 6063187D
 P 5800 6200
-F 0 "C15" H 5915 6246 50  0000 L CNN
+F 0 "C18" H 5915 6246 50  0000 L CNN
 F 1 "C" H 5915 6155 50  0000 L CNN
 F 2 "Capacitor_SMD:C_0805_2012Metric" H 5838 6050 50  0001 C CNN
@@
 Connection ~ 5800 6050
 $Comp
-L Device:C C16
+L Device:C C20
 U 1 1 606320AF
 P 6325 6200
-F 0 "C16" H 6440 6246 50  0000 L CNN
+F 0 "C20" H 6440 6246 50  0000 L CNN
 F 1 "C" H 6440 6155 50  0000 L CNN
 F 2 "Capacitor_SMD:C_0805_2012Metric" H 6363 6050 50  0001 C CNN
