File: pcb-using-pico/psion-org2-power/psion-org2-power_with_programming.sch (KiCad schematic (older format))
At the start: 25 parts, among them J1 Conn_02x08_Odd_Even, J2 Conn_02x08_Odd_Even, J3 Conn_01x27_Female, J4 Conn_02x08_Odd_Even, J5 Conn_01x11_Female, J6 Conn_01x02_Female, M1 P-CHANNEL-MOSFET, U1 ESP32-WROOM-32, U2 AMS1117-3.3, U3 CAT24C256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

Commit message: First layouts for fabrication
Parts:
- added C10, C4: 22uF, Capacitor_SMD:C_1210_3225Metric_Pad1.42x2.65mm_HandSolder, symbol Device:C_Small
- added C11, C12, C9: 100n, Capacitor_SMD:C_0805_2012Metric, symbol Device:C
- added C5: 1u, Capacitor_SMD:C_0805_2012Metric, symbol Device:C
- added D1: D, Diode_SMD:D_SOD-123, symbol Device:D
- added JP1: SolderJumper_2_Open, Jumper:SolderJumper-2_P1.3mm_Open_RoundedPad1.0x1.5mm, symbol Jumper:SolderJumper_2_Open
- added L1: 22uH, Inductor_SMD:L_Coilcraft_LPS5030, symbol pspice:INDUCTOR
- added M2: P-CHANNEL-MOSFET, Package_TO_SOT_SMD:SOT-23, symbol GeekAmmo:P-CHANNEL-MOSFET
- added M3: AO3401, Package_TO_SOT_SMD:SOT-23, symbol GeekAmmo:P-CHANNEL-MOSFET
- added R10: R_Small, Resistor_SMD:R_0805_2012Metric_Pad1.15x1.40mm_HandSolder, symbol Device:R_Small
- added R3: 120k, Resistor_SMD:R_0805_2012Metric_Pad1.15x1.40mm_HandSolder, symbol Device:R_Small
- added R4, R5: 18k, Resistor_SMD:R_0805_2012Metric_Pad1.15x1.40mm_HandSolder, symbol Device:R_Small
- added R8, R9: 100k, Resistor_SMD:R_0805_2012Metric_Pad1.15x1.40mm_HandSolder, symbol Device:R_Small
- added TR3, TR4, TR7, TR8: AO3400, Package_TO_SOT_SMD:SOT-23, symbol New_Library:Si2302CDS-n-channel
- added U8: Regulator_Switching_MT3608, Package_TO_SOT_SMD:SOT-23-6, symbol cq1re1-cache:Regulator_Switching_MT3608
Connections:
- net +3V3: now also C11.1, C12.1, C5.1, C9.1
- net GND: now also C10.2, C11.2, C12.2, C4.2, C5.2, C9.2, R9.2, TR3.2 (S), TR4.2 (S), TR7.2 (S), TR8.2 (S), U8.2 (GND)
- net VBAT_SWITCHED2: now also M2.2 (S), R8.1
- net VPP: now also M3.3 (D)
- net VPP_ON: now also TR7.1 (G)
- net VPP_SLOT_ON: now also TR8.1 (G)
- net VPP_X2: now reaches U5.1 (QB)
- net VPP_X2: now also TR4.1 (G)
- net VPP_X1: now reaches U5.15 (QA)
- net VPP_X1: now also TR3.1 (G)
- new net: R3.2, R4.1, R5.1, R9.1, U8.3 (FB)
- new net: R5.2, TR4.3 (D)
- new net: C4.1, L1.1, M2.3 (D), U8.4 (EN), U8.5 (IN)
- new net: C10.1, D1.1 (K), JP1.1 (A), R3.1
- new net: D1.2 (A), L1.2, U8.1 (SW)
- new net: JP1.2 (B), M3.2 (S), R10.1
- new net: M2.1 (G), R8.2, TR7.3 (D)
- new net: R4.2, TR3.3 (D)
- new net: M3.1 (G), R10.2, TR8.3 (D)
Other:
- note added: "Check values\n"
