File: pcb-using-pico/psion-org2-power/psion-org2-power.kicad_pcb (KiCad board)
At the start: 2 copper layers, 71.8 x 103.1 mm, 52 parts, among them J1 Conn_02x08_Odd_Even, J2 Conn_02x08_Odd_Even, J3 Conn_01x27_Female, J4 Conn_02x08_Odd_Even, J5 Conn_01x11_Female, J6 Conn_01x02_Female, J7 Conn_01x03_Female, M1 P-CHANNEL-MOSFET, M2 P-CHANNEL-MOSFET, U1 ESP32-WROOM-32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

Commit message: V1.1 PCBs
Parts:
- added J8: Conn_01x01_Female, ajm_kicad:psion_beeper_pad, B.Cu at (107.6, 44.9)
- added J9: Conn_01x01_Female, ajm_kicad:psion_beeper_pad, B.Cu at (125.8, 44.9)
- moved TR2 11.3 mm to (133.3, 34.7)
- moved R12 7.67 mm to (133.3, 37.7)
- moved R15 6.20 mm to (87.4, 59.8)
- moved U7 6.20 mm to (92.8, 56.8)
- moved M1 3.30 mm to (129.8, 39.3)
- moved C10 2.80 mm to (88.2, 55.8), turned to 270 degrees
- moved R4 0.20 mm to (98.3, 59.0)
Connections:
- J3 pad 14: (no net) -> BUZZER
Routing:
- net BUZZER: track 0.00 -> 82.1 mm, vias 0 -> 6
- net P_SPGM: track 106.4 -> 74.8 mm
- net EX_ON_INV: track 172.1 -> 193.2 mm, vias 5 -> 6
- net GND: track 444.1 -> 460.7 mm, vias 34 -> 38
- net LATCHOUT2: track 39.9 -> 55.0 mm, vias 4 -> 8
- net EX_ON: track 17.1 -> 31.7 mm
- net SC_OE: track 70.2 -> 80.5 mm
- net LS_DIR: track 43.9 -> 53.6 mm
- net P_SD4: track 120.8 -> 128.6 mm
- net SD6: track 30.1 -> 36.9 mm
- net SD7: track 34.0 -> 40.0 mm
- net SD4: track 23.4 -> 28.6 mm
- net PICO_TX: track 106.7 -> 111.2 mm
- net PICO_RX: track 105.8 -> 110.2 mm
- net EXT_PWR_IN: track 112.9 -> 117.0 mm
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Other:
- outline, holes or cut-outs redrawn

Commit message: fab2 V1.1
Routing:
- added copper zone on B.Cu, net GND
- added copper zone on F.Cu, net GND
Other:
- board text added: "RX"
- board text added: "TX"
- board text added: "WROOM PROG"
Changed lines of the file:
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@@
   (general
     (thickness 1.6)
-    (drawings 51)
+    (drawings 55)
     (tracks 3229)
     (zones 0)
@@
     (tags "Surface mounted pin header SMD 1x03 2.54mm single row style1 pin1 left")
     (attr smd)
-    (fp_text reference J7 (at 0 4.87 90) (layer B.SilkS)
+    (fp_text reference J7 (at 4.4 4.2 180) (layer B.SilkS)
       (effects (font (size 1 1) (thickness 0.15)) (justify mirror))
     )
@@
     )
   )
-  (gr_line (start 95.4 38.1) (end 129.6 38.1) (layer F.SilkS) (width 0.15))
+  (gr_line (start 129.6 38.1) (end 118.5 38.1) (layer F.SilkS) (width 0.15))
+  (gr_text RX (at 130.9 69.8) (layer B.SilkS)
+    (effects (font (size 1 1) (thickness 0.15)) (justify mirror))
+  )
+  (gr_text TX (at 136.9 69.9) (layer B.SilkS)
+    (effects (font (size 1 1) (thickness 0.15)) (justify mirror))
+  )
+  (gr_text GND (at 135.8 67.8) (layer B.SilkS)
+    (effects (font (size 1 1) (thickness 0.15)) (justify mirror))
+  )
+  (gr_text "WROOM\nPROG" (at 124.9 68) (layer B.SilkS)
+    (effects (font (size 1 1) (thickness 0.15)) (justify mirror))
+  )
   (gr_circle (center 89.9 34.425) (end 91.15 34.425) (layer Edge.Cuts) (width 0.1))
   (gr_circle (center 126.7 34.425) (end 127.95 34.425) (layer Edge.Cuts) (width 0.1))
@@
   (segment (start 85.845326 77.601493) (end 85.49339 77.953429) (width 0.25) (layer F.Cu) (net 62))
   (segment (start 90.268855 69.945861) (end 90.268855 70.870665) (width 0.25) (layer F.Cu) (net 62))
+  (zone (net 1) (net_name GND) (layer F.Cu) (hatch edge 0.508)
+    (connect_pads (clearance 0.508))
+    (min_thickness 0.254)
+    (fill yes (arc_segments 32) (thermal_gap 0.508) (thermal_bridge_width 0.508))
+    (polygon
+      (pts
+        (xy 150.4 26.5) (xy 156.8 132.9) (xy 77.7 133.1) (xy 76 24.6)
+      )
+    )
+  )
+  (zone (net 1) (net_name GND) (layer B.Cu) (hatch edge 0.508)
+    (connect_pads (clearance 0.508))
+    (min_thickness 0.254)
+    (fill yes (arc_segments 32) (thermal_gap 0.508) (thermal_bridge_width 0.508))
+    (polygon
+      (pts
+        (xy 150.6 26.1) (xy 158.5 134.4) (xy 76.2 134.4) (xy 76 133.6) (xy 74.7 23.4)
+      )
+    )
+  )
 )
