File: pcb-using-pico/psion-org2-power/psion-org2-power.kicad_pcb (KiCad board)
At the start: 2 copper layers, 71.8 x 103.1 mm, 54 parts, among them J1 Conn_02x08_Odd_Even, J2 Conn_02x08_Odd_Even, J3 Conn_01x27_Female, J4 Conn_02x08_Odd_Even, J5 Conn_01x11_Female, J6 Conn_01x02_Female, J7 Conn_01x03_Female, J8 Conn_01x01_Female, J9 Conn_01x01_Female, M1 P-CHANNEL-MOSFET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

Commit message: Updated missing values on schematics, pushed those through to the PCB and created BOM .csv files for those schematics. Created .pdf files for schematics to mitigate the missing library problem of Kicad 5.
Parts:
- C1, C2, C4, C5: value C_Small -> 100nF
- R1, R13, R14: value 100k -> 10k
- R2: value R_Small -> 10k
- R3: value R_Small -> 100k
Changed lines of the file:
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@@
     (add_net EX_ON_INV)
     (add_net GND)
+    (add_net LATCHOUT1)
     (add_net LATCHOUT2)
     (add_net LS_DIR)
     (add_net "Net-(C12-Pad1)")
     (add_net "Net-(D2-Pad2)")
+    (add_net "Net-(J2-Pad16)")
+    (add_net "Net-(J3-Pad16)")
+    (add_net "Net-(J4-Pad16)")
     (add_net "Net-(J7-Pad1)")
     (add_net "Net-(J7-Pad3)")
@@
     (add_net "Net-(R17-Pad2)")
     (add_net "Net-(R3-Pad1)")
+    (add_net "Net-(U1-Pad10)")
+    (add_net "Net-(U1-Pad11)")
+    (add_net "Net-(U1-Pad12)")
+    (add_net "Net-(U1-Pad13)")
+    (add_net "Net-(U1-Pad14)")
+    (add_net "Net-(U1-Pad16)")
+    (add_net "Net-(U1-Pad17)")
+    (add_net "Net-(U1-Pad18)")
+    (add_net "Net-(U1-Pad19)")
+    (add_net "Net-(U1-Pad20)")
+    (add_net "Net-(U1-Pad21)")
+    (add_net "Net-(U1-Pad22)")
+    (add_net "Net-(U1-Pad23)")
+    (add_net "Net-(U1-Pad24)")
+    (add_net "Net-(U1-Pad26)")
+    (add_net "Net-(U1-Pad29)")
+    (add_net "Net-(U1-Pad30)")
+    (add_net "Net-(U1-Pad31)")
+    (add_net "Net-(U1-Pad32)")
+    (add_net "Net-(U1-Pad33)")
+    (add_net "Net-(U1-Pad36)")
+    (add_net "Net-(U1-Pad37)")
+    (add_net "Net-(U1-Pad4)")
+    (add_net "Net-(U1-Pad5)")
+    (add_net "Net-(U1-Pad6)")
+    (add_net "Net-(U1-Pad7)")
+    (add_net "Net-(U1-Pad8)")
+    (add_net "Net-(U1-Pad9)")
+    (add_net "Net-(U5-Pad1)")
+    (add_net "Net-(U5-Pad15)")
+    (add_net "Net-(U5-Pad2)")
+    (add_net "Net-(U5-Pad6)")
+    (add_net "Net-(U5-Pad7)")
+    (add_net "Net-(U5-Pad9)")
+    (add_net "Net-(U6-Pad11)")
     (add_net OLED_SCL)
     (add_net OLED_SDA)
@@
     (add_net SD6)
     (add_net SD7)
+    (add_net SDAOUT)
     (add_net SD_OE)
     (add_net SMR)
@@
     (add_net SS3)
     (add_net VBAT)
+    (add_net VBAT_SWITCHED1)
     (add_net VBAT_SWITCHED2)
     (add_net VCC_ESP)
@@
       (effects (font (size 1 1) (thickness 0.15)))
     )
-    (fp_text value 100k (at 0 1.65 90) (layer F.Fab)
+    (fp_text value 10k (at 0 1.65 90) (layer F.Fab)
       (effects (font (size 1 1) (thickness 0.15)))
     )
@@
       (effects (font (size 1 1) (thickness 0.15)))
     )
-    (fp_text value 100k (at 0 1.65) (layer F.Fab)
+    (fp_text value 10k (at 0 1.65) (layer F.Fab)
       (effects (font (size 1 1) (thickness 0.15)))
     )
@@
       (effects (font (size 1 1) (thickness 0.15)))
     )
-    (fp_text value R_Small (at 0 1.65 90) (layer F.Fab)
+    (fp_text value 100k (at 0 1.65 90) (layer F.Fab)
       (effects (font (size 1 1) (thickness 0.15)))
     )
@@
       (effects (font (size 1 1) (thickness 0.15)))
     )
-    (fp_text value C_Small (at 0 1.65 90) (layer F.Fab)
+    (fp_text value 100nF (at 0 1.65 90) (layer F.Fab)
       (effects (font (size 1 1) (thickness 0.15)))
     )
@@
       (effects (font (size 1 1) (thickness 0.15)))
     )
-    (fp_text value C_Small (at 0 1.65) (layer F.Fab)
+    (fp_text value 100nF (at 0 1.65) (layer F.Fab)
       (effects (font (size 1 1) (thickness 0.15)))
     )
@@
       (effects (font (size 1 1) (thickness 0.15)))
     )
-    (fp_text value 100k (at 0 1.65) (layer F.Fab)
+    (fp_text value 10k (at 0 1.65) (layer F.Fab)
       (effects (font (size 1 1) (thickness 0.15)))
     )
@@
       (effects (font (size 1 1) (thickness 0.15)))
     )
-    (fp_text value R_Small (at 0 1.65 90) (layer F.Fab)
+    (fp_text value 10k (at 0 1.65 90) (layer F.Fab)
       (effects (font (size 1 1) (thickness 0.15)))
     )
@@
       (effects (font (size 1 1) (thickness 0.15)))
     )
-    (fp_text value C_Small (at 0 1.65 90) (layer F.Fab)
+    (fp_text value 100nF (at 0 1.65 90) (layer F.Fab)
       (effects (font (size 1 1) (thickness 0.15)))
     )
@@
       (effects (font (size 1 1) (thickness 0.15)))
     )
-    (fp_text value C_Small (at 0 1.65 90) (layer F.Fab)
-      (effects (font (size 1 1) (thickness 0.15)))
-    )
+    (fp_text value 100nF (at 0 1.65 90) (layer F.Fab)
+      (effects (font (size 1 1) (thickness 0.15)))
+    )
