File: pcb_using_pico_w/psion-org2-power/file612F7BBD.sch (KiCad schematic (older format))
At the start: 39 parts, among them SW1 AC_ON, SW10 n, SW11 t, SW12 del, SW13 up, SW14 c, SW15 i, SW16 o, SW17 u, SW18 y, SW19 down, SW2 A, SW20 d, SW21 j, SW22 p, SW23 v, SW24 z, SW25 left, SW26 e, SW27 k, SW28 q, SW29 w, SW3 g, SW30 spc, SW31 right, SW32 f, SW33 L, SW34 r, SW35 x, SW36 exe, SW4 m, SW5 s, SW6 shft, SW7 mode, SW8 b, SW9 h

Commit message: Added power board with VPP 21V supply
Parts:
- removed D?: 2v7, Diode_SMD:D_SOD-123, symbol Device:D
- removed R?: nopop, Resistor_SMD:R_0805_2012Metric, symbol Device:R_Small
- removed R?: 2k2, Resistor_SMD:R_0805_2012Metric, symbol Device:R_Small
Connections:
- net K3: now also SW7.2 (B)
- net K4: now also SW13.2 (B)
- net K5: now also SW25.2 (B)
- net K6: now also SW31.2 (B)
- net K7: now also SW19.2 (B)
- net P52: no longer SW7.2 (B)
- net P54: no longer SW19.2 (B)
- net P55: no longer SW25.2 (B)
- net P56: no longer SW31.2 (B)
- net P57: now also SW1.2 (B)
- net P53 renamed p53
- net p53: no longer SW13.2 (B)
- net VBAT renamed +3V3
